File: Bomba_Javi/Bomba.sch (EAGLE design)
At the start: 3 parts, among them IC1 PIC12F629SN, K1 G5LE

Commit message: Pcb continuado
Parts:
- removed JP1: (no value), SparkFun-Connectors:M025MM
- added 5V, BOTON: (no value), SparkFun-Connectors:M025MM
- added D1: (no value), SparkFun-DiscreteSemi:DIODE1N4148
- added ISP: (no value), SparkFun-Connectors:M05LOCK_LONGPADS
- added Q1: (no value), SparkFun-DiscreteSemi:TRANSISTOR_NPNSOT23
- added R1, R2: (no value), SparkFun-Passives:RESISTOR1206
- added R3: 1k, SparkFun-Passives:RESISTOR1206
Connections:
- new net 5V: 5V.2, IC1.VDD, Q1.C
- new net A: IC1.GP3, R3.2
- new net GND: 5V.1, BOTON.1, D1.A, IC1.VSS, K11.2
- new net N$2: D1.C, K11.1, Q1.E
- new net N$3: BOTON.2, IC1.GP2
- new net N$4: Q1.B, R3.1
Other:
- moved on the sheet: K1
Changed lines of the file:
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@@
 <parts>
 <part name="IC1" library="microchip" deviceset="PIC12F6*" device="SN" technology="29"/>
-<part name="JP1" library="SparkFun-Connectors" deviceset="M02" device="5MM"/>
+<part name="5V" library="SparkFun-Connectors" deviceset="M02" device="5MM"/>
 <part name="K1" library="relay" deviceset="G5LE" device=""/>
+<part name="BOTON" library="SparkFun-Connectors" deviceset="M02" device="5MM"/>
+<part name="U$1" library="SparkFun-Aesthetics" deviceset="5V" device=""/>
+<part name="GND1" library="SparkFun-Aesthetics" deviceset="GND" device=""/>
+<part name="U$2" library="SparkFun-Aesthetics" deviceset="5V" device=""/>
+<part name="GND2" library="SparkFun-Aesthetics" deviceset="GND" device=""/>
+<part name="Q1" library="SparkFun-DiscreteSemi" deviceset="TRANSISTOR_NPN" device="SOT23"/>
+<part name="D1" library="SparkFun-DiscreteSemi" deviceset="DIODE" device="1N4148"/>
+<part name="R1" library="SparkFun-Passives" deviceset="RESISTOR" device="1206"/>
+<part name="R2" library="SparkFun-Passives" deviceset="RESISTOR" device="1206"/>
+<part name="R3" library="SparkFun-Passives" deviceset="RESISTOR" device="1206" value="1k"/>
+<part name="GND3" library="SparkFun-Aesthetics" deviceset="GND" device=""/>
+<part name="ISP" library="SparkFun-Connectors" deviceset="M05" device="LOCK_LONGPADS"/>
+<part name="U$3" library="SparkFun-Aesthetics" deviceset="5V" device=""/>
+<part name="GND4" library="SparkFun-Aesthetics" deviceset="GND" device=""/>
 </parts>
 <sheets>
@@
 <instances>
 <instance part="IC1" gate="G$1" x="63.5" y="63.5"/>
-<instance part="JP1" gate="G$1" x="5.08" y="33.02"/>
-<instance part="K1" gate="1" x="73.66" y="25.4"/>
-<instance part="K1" gate="2" x="96.52" y="25.4"/>
+<instance part="5V" gate="G$1" x="5.08" y="55.88"/>
+<instance part="K1" gate="1" x="119.38" y="60.96"/>
+<instance part="K1" gate="2" x="167.64" y="58.42"/>
+<instance part="BOTON" gate="G$1" x="96.52" y="55.88" rot="MR0"/>
+<instance part="U$1" gate="G$1" x="17.78" y="60.96"/>
+<instance part="GND1" gate="1" x="17.78" y="53.34"/>
+<instance part="U$2" gate="G$1" x="63.5" y="81.28"/>
+<instance part="GND2" gate="1" x="66.04" y="45.72"/>
+<instance part="Q1" gate="G$1" x="111.76" y="81.28"/>
+<instance part="D1" gate="G$1" x="109.22" y="60.96" rot="R90"/>
+<instance part="R1" gate="G$1" x="45.72" y="-5.08"/>
+<instance part="R2" gate="G$1" x="40.64" y="5.08"/>
+<instance part="R3" gate="G$1" x="96.52" y="81.28" rot="R180"/>
+<instance part="GND3" gate="1" x="83.82" y="50.8"/>
+<instance part="ISP" gate="G$1" x="5.08" y="83.82" rot="MR180"/>
+<instance part="U$3" gate="G$1" x="114.3" y="88.9"/>
+<instance part="GND4" gate="1" x="114.3" y="40.64"/>
 </instances>
 <busses>
 </busses>
 <nets>
+<net name="5V" class="0">
+<segment>
+<pinref part="5V" gate="G$1" pin="2"/>
+<pinref part="U$1" gate="G$1" pin="5V"/>
+<wire x1="12.7" y1="58.42" x2="17.78" y2="58.42" width="0.1524" layer="91"/>
+<wire x1="17.78" y1="58.42" x2="17.78" y2="60.96" width="0.1524" layer="91"/>
+</segment>
+<segment>
+<pinref part="U$2" gate="G$1" pin="5V"/>
+<pinref part="IC1" gate="G$1" pin="VDD"/>
+<wire x1="63.5" y1="81.28" x2="63.5" y2="76.2" width="0.1524" layer="91"/>
+</segment>
+<segment>
+<pinref part="U$3" gate="G$1" pin="5V"/>
+<pinref part="Q1" gate="G$1" pin="C"/>
+<wire x1="114.3" y1="88.9" x2="114.3" y2="86.36" width="0.1524" layer="91"/>
+</segment>
+</net>
+<net name="GND" class="0">
+<segment>
+<pinref part="5V" gate="G$1" pin="1"/>
+<pinref part="GND1" gate="1" pin="GND"/>
+<wire x1="12.7" y1="55.88" x2="17.78" y2="55.88" width="0.1524" layer="91"/>
+</segment>
+<segment>
+<pinref part="GND2" gate="1" pin="GND"/>
+<pinref part="IC1" gate="G$1" pin="VSS"/>
+<wire x1="66.04" y1="48.26" x2="66.04" y2="53.34" width="0.1524" layer="91"/>
+</segment>
+<segment>
+<pinref part="BOTON" gate="G$1" pin="1"/>
+<pinref part="GND3" gate="1" pin="GND"/>
+<wire x1="88.9" y1="55.88" x2="83.82" y2="55.88" width="0.1524" layer="91"/>
+<wire x1="83.82" y1="55.88" x2="83.82" y2="53.34" width="0.1524" layer="91"/>
+</segment>
+<segment>
+<pinref part="D1" gate="G$1" pin="A"/>
+<wire x1="109.22" y1="58.42" x2="109.22" y2="45.72" width="0.1524" layer="91"/>
+<wire x1="109.22" y1="45.72" x2="114.3" y2="45.72" width="0.1524" layer="91"/>
+<pinref part="K1" gate="1" pin="2"/>
+<wire x1="114.3" y1="45.72" x2="119.38" y2="45.72" width="0.1524" layer="91"/>
+<wire x1="119.38" y1="45.72" x2="119.38" y2="55.88" width="0.1524" layer="91"/>
+<pinref part="GND4" gate="1" pin="GND"/>
+<wire x1="114.3" y1="43.18" x2="114.3" y2="45.72" width="0.1524" layer="91"/>
+</segment>
+</net>
+<net name="N$2" class="0">
+<segment>
+<pinref part="D1" gate="G$1" pin="C"/>
+<wire x1="109.22" y1="63.5" x2="109.22" y2="71.12" width="0.1524" layer="91"/>
+<wire x1="109.22" y1="71.12" x2="114.3" y2="71.12" width="0.1524" layer="91"/>
+<pinref part="K1" gate="1" pin="1"/>
+<wire x1="114.3" y1="71.12" x2="119.38" y2="71.12" width="0.1524" layer="91"/>
+<wire x1="119.38" y1="71.12" x2="119.38" y2="66.04" width="0.1524" layer="91"/>
+<pinref part="Q1" gate="G$1" pin="E"/>
+<wire x1="114.3" y1="76.2" x2="114.3" y2="71.12" width="0.1524" layer="91"/>
+</segment>
+</net>
+<net name="N$3" class="0">
+<segment>
+<pinref part="IC1" gate="G$1" pin="GP2"/>
+<wire x1="78.74" y1="60.96" x2="88.9" y2="60.96" width="0.1524" layer="91"/>
+<pinref part="BOTON" gate="G$1" pin="2"/>
+<wire x1="88.9" y1="60.96" x2="88.9" y2="58.42" width="0.1524" layer="91"/>
+</segment>
+</net>
+<net name="N$4" class="0">
+<segment>
+<pinref part="R3" gate="G$1" pin="1"/>
+<pinref part="Q1" gate="G$1" pin="B"/>
+<wire x1="101.6" y1="81.28" x2="109.22" y2="81.28" width="0.1524" layer="91"/>
+</segment>
+</net>
+<net name="A" class="0">
+<segment>
+<pinref part="IC1" gate="G$1" pin="GP3"/>
+<wire x1="50.8" y1="58.42" x2="43.18" y2="58.42" width="0.1524" layer="91"/>
+<label x="43.18" y="58.42" size="1.778" layer="95"/>
+</segment>
+<segment>
+<pinref part="R3" gate="G$1" pin="2"/>
+<wire x1="91.44" y1="81.28" x2="81.28" y2="81.28" width="0.1524" layer="91"/>
+<label x="83.82" y="81.28" size="1.778" layer="95"/>
+</segment>
+</net>
 </nets>
 </sheet>

Commit message: Pcb continuado
Parts:
- added C1: (no value), SparkFun-Passives:CAP_POLPTH1
- added LED: (no value), SparkFun-Connectors:M02LOCK_LONGPADS
- added LUZ: (no value), SparkFun-Connectors:M025MM
- R1: value (none) -> 1K
- R2: value (none) -> 10k
Connections:
- new net N$6: K12.S, LUZ.2
- new net N$7: K12.P, LUZ.1
- new net N$8: IC1.GP5/CLKIN, R1.2
- new net N$9: LED.2, R1.1
- new net PGC: IC1.GP1, ISP.5
- new net PGD: IC1.GP0, ISP.4
- new net RST: IC1.GP3, ISP.1, R2.1
- net 5V: now also C1.+, ISP.2, R2.2
- net A: now also IC1.GP4/CLKOUT; no longer IC1.GP3
- net GND: now also C1.-, ISP.3, LED.1
Other:
- moved on the sheet: R1, R2
