File: Bomba_Javi/Bomba.brd (EAGLE design)
At the start: 3 parts, among them IC1 PIC12F629SN, K1 G5LE

Commit message: Pcb continuado
Parts:
- removed JP1: (no value), SparkFun-Connectors:SCREWTERMINAL-5MM-2
- added 5V, BOTON: (no value), SparkFun-Connectors:SCREWTERMINAL-5MM-2
- added D1: (no value), SparkFun-DiscreteSemi:DIODE-1N4148
- added ISP: (no value), SparkFun-Connectors:1X05_LOCK_LONGPADS
- added Q1: (no value), SparkFun-DiscreteSemi:SOT23
- added R1, R2: (no value), SparkFun-Passives:1206
- added R3: 1k, SparkFun-Passives:1206
Connections:
- removed net VDD: IC1.1
- removed net VSS: IC1.8
- new net 5V: 5V.2, IC1.1, Q1.3
- new net A: IC1.4, R3.2
- new net GND: 5V.1, BOTON.1, D1.A, IC1.8, K1.2
- new net N$2: D1.C, K1.1, Q1.2
- new net N$3: BOTON.2, IC1.5
- new net N$4: Q1.1, R3.1
Changed lines of the file:
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@@
 <attribute name="OC_FARNELL" value="9759000" x="11.43" y="8.89" size="1.778" layer="27" display="off"/>
 </element>
-<element name="JP1" library="SparkFun-Connectors" package="SCREWTERMINAL-5MM-2" value="" x="11.43" y="0"/>
+<element name="5V" library="SparkFun-Connectors" package="SCREWTERMINAL-5MM-2" value="" x="45.72" y="38.1"/>
 <element name="K1" library="relay" package="G5LE" value="G5LE" x="41.91" y="11.43">
 <attribute name="OC_NEWARK" value="unknown" x="41.91" y="11.43" size="1.778" layer="27" display="off"/>
@@
 <attribute name="OC_FARNELL" value="unknown" x="41.91" y="11.43" size="1.778" layer="27" display="off"/>
 </element>
+<element name="BOTON" library="SparkFun-Connectors" package="SCREWTERMINAL-5MM-2" value="" x="26.67" y="26.67"/>
+<element name="Q1" library="SparkFun-DiscreteSemi" package="SOT23" value="" x="43.18" y="27.94"/>
+<element name="D1" library="SparkFun-DiscreteSemi" package="DIODE-1N4148" value="" x="53.34" y="25.4"/>
+<element name="R1" library="SparkFun-Passives" package="1206" value="" x="59.69" y="20.32"/>
+<element name="R2" library="SparkFun-Passives" package="1206" value="" x="13.97" y="20.32"/>
+<element name="R3" library="SparkFun-Passives" package="1206" value="1k" x="16.51" y="26.67"/>
+<element name="ISP" library="SparkFun-Connectors" package="1X05_LOCK_LONGPADS" value="" x="8.89" y="-1.27"/>
 </elements>
 <signals>
-<signal name="VDD">
+<signal name="5V">
+<contactref element="5V" pad="2"/>
 <contactref element="IC1" pad="1"/>
+<contactref element="Q1" pad="3"/>
+<wire x1="43.18" y1="29.04" x2="50.72" y2="38.1" width="0" layer="19" extent="1-1"/>
+<wire x1="9.525" y1="6.29" x2="43.18" y2="29.04" width="0" layer="19" extent="1-1"/>
 </signal>
-<signal name="VSS">
+<signal name="GND">
+<contactref element="5V" pad="1"/>
 <contactref element="IC1" pad="8"/>
+<contactref element="BOTON" pad="1"/>
+<contactref element="D1" pad="A"/>
+<contactref element="K1" pad="2"/>
+<wire x1="49.53" y1="25.4" x2="45.72" y2="38.1" width="0" layer="19" extent="1-1"/>
+<wire x1="34.417" y1="17.399" x2="49.53" y2="25.4" width="0" layer="19" extent="1-1"/>
+<wire x1="26.67" y1="26.67" x2="34.417" y2="17.399" width="0" layer="19" extent="1-1"/>
+<wire x1="9.525" y1="11.49" x2="26.67" y2="26.67" width="0" layer="19" extent="1-1"/>
+</signal>
+<signal name="N$2">
+<contactref element="D1" pad="C"/>
+<contactref element="K1" pad="1"/>
+<contactref element="Q1" pad="2"/>
+<wire x1="44.13" y1="26.84" x2="57.15" y2="25.4" width="0" layer="19" extent="1-1"/>
+<wire x1="34.417" y1="5.461" x2="44.13" y2="26.84" width="0" layer="19" extent="1-1"/>
+</signal>
+<signal name="N$3">
+<contactref element="IC1" pad="5"/>
+<contactref element="BOTON" pad="2"/>
+<wire x1="13.335" y1="11.49" x2="31.67" y2="26.67" width="0" layer="19" extent="1-1"/>
+</signal>
+<signal name="N$4">
+<contactref element="R3" pad="1"/>
+<contactref element="Q1" pad="1"/>
+<wire x1="15.11" y1="26.67" x2="42.23" y2="26.84" width="0" layer="19" extent="1-1"/>
+</signal>
+<signal name="A">
+<contactref element="IC1" pad="4"/>
+<contactref element="R3" pad="2"/>
+<wire x1="13.335" y1="6.29" x2="17.91" y2="26.67" width="0" layer="19" extent="1-1"/>
 </signal>
 </signals>

Commit message: Pcb continuado
Parts:
- added C1: (no value), SparkFun-Passives:CPOL-RADIAL-100UF-25V
- added LED: (no value), SparkFun-Connectors:1X02_LOCK_LONGPADS
- added LUZ: (no value), SparkFun-Connectors:SCREWTERMINAL-5MM-2
- R1: value (none) -> 1K
- R2: value (none) -> 10k
- moved IC1 48.6 mm to (52.1, 35.6), flipped to the bottom, turned to 270 degrees
- moved K1 47.6 mm to (81.3, 38.1)
- moved R3 44.0 mm to (59.8, 34.3), flipped to the bottom
- moved R2 40.5 mm to (53.3, 29.7), flipped to the bottom
- moved ISP 37.7 mm to (40.6, 19.1), turned to 90 degrees
- moved BOTON 28.7 mm to (54.6, 20.3), flipped to the bottom
- moved Q1 19.1 mm to (62.2, 29.2), flipped to the bottom, turned to 180 degrees
- moved D1 18.0 mm to (66.0, 38.1), turned to 270 degrees
- moved R1 16.5 mm to (59.8, 36.8), flipped to the bottom
- moved 5V 6.84 mm to (39.4, 35.6), turned to 90 degrees
Connections:
- new net N$6: K1.S, LUZ.2
- new net N$7: K1.P, LUZ.1
- new net N$8: IC1.2, R1.2
- new net N$9: LED.2, R1.1
- new net PGC: IC1.6, ISP.5
- new net PGD: IC1.7, ISP.4
- new net RST: IC1.4, ISP.1, R2.1
- net 5V: now also C1.1, ISP.2, R2.2
- net A: now also IC1.3; no longer IC1.4
- net GND: now also C1.2, ISP.3, LED.1
Routing:
- net RST: track 0.00 -> 28.2 mm
- net N$7: track 0.00 -> 24.9 mm
- net PGD: track 0.00 -> 22.1 mm
- net N$2: track 0.00 -> 13.9 mm
- net N$6: track 0.00 -> 12.7 mm
- net PGC: track 0.00 -> 11.2 mm
- net GND: track 0.00 -> 8.79 mm
- net N$9: track 0.00 -> 5.21 mm
- net A: track 0.00 -> 4.90 mm
- net N$8: track 0.00 -> 4.89 mm
- net N$4: track 0.00 -> 4.01 mm

Commit message: PCB terminado. PDF
Routing:
- net GND: track 8.79 -> 117.2 mm
- net 5V: track 0.00 -> 73.0 mm, vias 0 -> 3
- net N$3: track 0.00 -> 13.5 mm
- added copper zone on layer 16, net GND
Changed lines of the file:
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@@
 <contactref element="R2" pad="2"/>
 <contactref element="C1" pad="1"/>
-<wire x1="54.67" y1="37.465" x2="53.213" y2="40.64" width="0" layer="19" extent="16-16"/>
-<wire x1="51.94" y1="29.718" x2="54.67" y2="37.465" width="0" layer="19" extent="16-16"/>
-<wire x1="62.23" y1="28.11" x2="51.94" y2="29.718" width="0" layer="19" extent="16-16"/>
-<wire x1="40.894" y1="21.59" x2="51.94" y2="29.718" width="0" layer="19" extent="16-16"/>
-<wire x1="39.37" y1="40.56" x2="53.213" y2="40.64" width="0" layer="19" extent="1-1"/>
+<wire x1="54.67" y1="37.465" x2="54.102" y2="37.465" width="0.6096" layer="16"/>
+<wire x1="54.102" y1="37.465" x2="53.4035" y2="38.1635" width="0.6096" layer="16"/>
+<wire x1="53.4035" y1="38.1635" x2="53.34" y2="38.227" width="0.6096" layer="16"/>
+<wire x1="53.34" y1="38.227" x2="53.34" y2="40.513" width="0.6096" layer="16"/>
+<wire x1="53.34" y1="40.513" x2="53.213" y2="40.64" width="0.6096" layer="16"/>
+<wire x1="51.94" y1="29.718" x2="51.94" y2="36.7" width="0.6096" layer="16"/>
+<wire x1="51.94" y1="36.7" x2="53.4035" y2="38.1635" width="0.6096" layer="16"/>
+<wire x1="39.37" y1="40.56" x2="39.37" y2="40.64" width="1.27" layer="16"/>
+<wire x1="39.37" y1="40.64" x2="41.91" y2="43.18" width="1.27" layer="16"/>
+<wire x1="41.91" y1="43.18" x2="44.45" y2="43.18" width="1.27" layer="16"/>
+<wire x1="44.45" y1="43.18" x2="45.72" y2="43.18" width="1.27" layer="16"/>
+<wire x1="45.72" y1="43.18" x2="51.562" y2="43.18" width="1.27" layer="16"/>
+<wire x1="51.562" y1="43.18" x2="53.213" y2="41.529" width="1.27" layer="16"/>
+<wire x1="53.213" y1="41.529" x2="53.213" y2="40.64" width="1.27" layer="16"/>
+<wire x1="62.23" y1="28.11" x2="59.52" y2="28.11" width="1.016" layer="16"/>
+<wire x1="59.52" y1="28.11" x2="58.166" y2="29.845" width="1.016" layer="16"/>
+<via x="58.166" y="29.845" extent="1-16" drill="1" diameter="2.54"/>
+<via x="45.72" y="43.18" extent="1-16" drill="1" diameter="2.54"/>
+<via x="45.72" y="29.21" extent="1-16" drill="1" diameter="2.54"/>
+<wire x1="45.72" y1="29.21" x2="57.531" y2="29.21" width="1.016" layer="1"/>
+<wire x1="57.531" y1="29.21" x2="58.166" y2="29.845" width="1.016" layer="1"/>
+<wire x1="45.72" y1="29.21" x2="45.72" y2="43.18" width="1.016" layer="1"/>
+<wire x1="40.894" y1="21.59" x2="44.45" y2="21.59" width="1.016" layer="16"/>
+<wire x1="44.45" y1="21.59" x2="45.72" y2="22.86" width="1.016" layer="16"/>
+<wire x1="45.72" y1="22.86" x2="45.72" y2="29.21" width="1.016" layer="16"/>
 </signal>
 <signal name="GND">
@@
 <wire x1="66.04" y1="42.164" x2="67.945" y2="44.069" width="1.27" layer="16"/>
 <wire x1="67.945" y1="44.069" x2="73.787" y2="44.069" width="1.27" layer="16"/>
-<wire x1="58.293" y1="41.91" x2="66.04" y2="41.91" width="0" layer="19" extent="1-1"/>
-<wire x1="50.673" y1="40.64" x2="58.293" y2="41.91" width="0" layer="19" extent="1-1"/>
-<wire x1="49.47" y1="37.465" x2="50.673" y2="40.64" width="0" layer="19" extent="16-16"/>
-<wire x1="39.37" y1="35.56" x2="49.47" y2="37.465" width="0" layer="19" extent="16-16"/>
-<wire x1="40.64" y1="24.13" x2="39.37" y2="35.56" width="0" layer="19" extent="1-1"/>
-<wire x1="54.61" y1="20.32" x2="40.64" y2="24.13" width="0" layer="19" extent="1-1"/>
+<wire x1="49.47" y1="37.465" x2="49.657" y2="37.465" width="0.6096" layer="16"/>
+<wire x1="49.657" y1="37.465" x2="50.673" y2="38.481" width="0.6096" layer="16"/>
+<wire x1="50.673" y1="38.481" x2="50.673" y2="40.64" width="0.6096" layer="16"/>
+<wire x1="49.47" y1="37.465" x2="41.275" y2="37.465" width="0.6096" layer="16"/>
+<wire x1="41.275" y1="37.465" x2="39.37" y2="35.56" width="0.6096" layer="16"/>
+<wire x1="39.37" y1="35.56" x2="36.83" y2="35.56" width="1.27" layer="16"/>
+<wire x1="36.83" y1="35.56" x2="34.29" y2="33.02" width="1.27" layer="16"/>
+<wire x1="34.29" y1="33.02" x2="34.29" y2="26.67" width="1.27" layer="16"/>
+<wire x1="34.29" y1="26.67" x2="36.83" y2="24.13" width="1.27" layer="16"/>
+<wire x1="36.83" y1="24.13" x2="40.64" y2="24.13" width="1.27" layer="16"/>
+<wire x1="58.293" y1="41.91" x2="58.293" y2="44.323" width="1.27" layer="16"/>
+<wire x1="58.293" y1="44.323" x2="59.69" y2="45.72" width="1.27" layer="16"/>
+<wire x1="59.69" y1="45.72" x2="62.23" y2="45.72" width="1.27" layer="16"/>
+<wire x1="62.23" y1="45.72" x2="66.04" y2="41.91" width="1.27" layer="16"/>
+<wire x1="58.293" y1="41.91" x2="58.293" y2="43.307" width="0.8128" layer="16"/>
+<wire x1="58.293" y1="43.307" x2="55.88" y2="45.72" width="0.8128" layer="16"/>
+<wire x1="55.88" y1="45.72" x2="39.37" y2="45.72" width="0.8128" layer="16"/>
+<wire x1="39.37" y1="45.72" x2="36.83" y2="43.18" width="0.8128" layer="16"/>
+<wire x1="36.83" y1="43.18" x2="36.83" y2="35.56" width="0.8128" layer="16"/>
+<wire x1="54.61" y1="20.32" x2="54.61" y2="17.78" width="1.016" layer="16"/>
+<wire x1="54.61" y1="17.78" x2="52.07" y2="15.24" width="1.016" layer="16"/>
+<wire x1="52.07" y1="15.24" x2="38.989" y2="15.24" width="1.016" layer="16"/>
+<wire x1="38.989" y1="15.24" x2="37.084" y2="17.145" width="1.016" layer="16"/>
+<wire x1="37.084" y1="17.145" x2="37.084" y2="23.876" width="1.016" layer="16"/>
+<wire x1="37.084" y1="23.876" x2="36.83" y2="24.13" width="1.016" layer="16"/>
+<polygon width="0.6096" layer="16" isolate="0.4064">
+<vertex x="66.5" y="46.228"/>
+<vertex x="66.5" y="15"/>
+<vertex x="33.782" y="15"/>
+<vertex x="33.782" y="46.228"/>
+</polygon>
 </signal>
 <signal name="N$2">
@@
 <contactref element="IC1" pad="5"/>
 <contactref element="BOTON" pad="2"/>
-<wire x1="49.61" y1="20.32" x2="49.47" y2="33.655" width="0" layer="19" extent="16-16"/>
+<wire x1="49.61" y1="20.32" x2="49.53" y2="20.32" width="1.27" layer="16"/>
+<wire x1="49.53" y1="20.32" x2="49.53" y2="33.02" width="1.27" layer="16"/>
+<wire x1="49.53" y1="33.02" x2="49.47" y2="33.02" width="0.6096" layer="16"/>
+<wire x1="49.47" y1="33.02" x2="49.47" y2="33.655" width="0.6096" layer="16"/>
 </signal>
 <signal name="N$4">
